Commit message: robot setup stable

File: erl_assignment_3_robot/urdf/robot.xacro (robot description, xacro)
@@ -171,12 +171,12 @@
 	    <child link="hokuyo_link"/>
 	 </joint>
-	   <link name="camera_link">
+	<link name="camera_link">
 	    <collision>
 	      <origin xyz="0 0 0.025" rpy="0 0 0"/>
-	      <geometry>
-		<box size="0.05 0.05 0.05"/>
-	      </geometry>
+	    <geometry>
+		<box size="0.05 0.05 0.05"/>
+	    </geometry> -->
 	    </collision>
-	    <visual>
+	    <!-- <visual>
 	      <origin xyz="0 0 0.025" rpy="0 0 0"/>
 	      <geometry>
@@ -186,5 +186,5 @@
 		<color rgba="1 0 0 1"/>
 	      </material>
-	    </visual>
+	    </visual>-->
 	    <inertial>
 	      <mass value="1e-5" />
@@ -195,5 +195,5 @@
   <joint name="camera_joint" type="fixed">
 	    <axis xyz="0 1 0" />
-	    <origin xyz="0.23 0 0.0" rpy="0 0 0"/>
+	    <origin xyz="0.23 0 0.25" rpy="0 0 0"/>
 	    <parent link="link_chassis"/>
 	    <child link="camera_link"/>
