Commit message: erl3 robot first setup

File: erl_assignment_3_robot/urdf/detectibot/detectibot.urdf (robot description, URDF)
Before this commit: robot robot2_laser_xacro, 4 links, 3 joints
Links:
- removed link link_left_wheel
- removed link link_right_wheel
- added link camera_link, mass 1e-5; collision box size=0.05 0.05 0.05; visual box size=0.05 0.05 0.05
- added link link_back_left_wheel, mass 0.2; collision cylinder length=0.04 radius=0.1; visual cylinder length=0.04 radius=0.1
- added link link_back_right_wheel, mass 0.2; collision cylinder length=0.04 radius=0.1; visual cylinder length=0.04 radius=0.1
- added link link_front_left_wheel, mass 0.2; collision cylinder length=0.04 radius=0.1; visual cylinder length=0.04 radius=0.1
- added link link_front_right_wheel, mass 0.2; collision cylinder length=0.04 radius=0.1; visual cylinder length=0.04 radius=0.1
- link link_chassis: geometry collision box size=0.5 0.3 0.07; visual box size=0.5 0.3 0.07
Joints:
- removed joint joint_left_wheel
- removed joint joint_right_wheel
- added joint camera_joint: type fixed, parent link_chassis, child camera_link, origin xyz=0.23 0 0.0 rpy=0 0 0, axis 0 1 0
- added joint joint_back_left_wheel: type continuous, parent link_chassis, child link_back_left_wheel, origin xyz=-0.20 -0.15 0 rpy=0 0 0, axis 0 1 0, limit effort=10000 velocity=1000
- added joint joint_back_right_wheel: type continuous, parent link_chassis, child link_back_right_wheel, origin xyz=-0.20 0.15 0 rpy=0 0 0, axis 0 1 0, limit effort=10000 velocity=1000
- added joint joint_front_left_wheel: type continuous, parent link_chassis, child link_front_left_wheel, origin xyz=0.20 -0.15 0 rpy=0 0 0, axis 0 1 0, limit effort=10000 velocity=1000
- added joint joint_front_right_wheel: type continuous, parent link_chassis, child link_front_right_wheel, origin xyz=0.20 0.15 0 rpy=0 0 0, axis 0 1 0, limit effort=10000 velocity=1000

Commit message: stable

File: erl_assignment_3_robot/urdf/detectibot/detectibot.urdf (robot description, URDF)
Before this commit: robot detectibot, 7 links, 6 joints
Links:
- link camera_link: geometry collision box size=0.05 0.05 0.05
Joints:
- joint camera_joint: origin xyz=0.23 0 0.0 rpy=0 0 0 -> xyz=0.23 0 0.25 rpy=0 0 0
